File: hardware/PortableLinuxGamestation.sch (EAGLE design)
At the start: 21 parts, among them U1 OSD3358-512M-BSM, Y1 ABS07-32.768KHZ-T, Y2 24MHz

Commit message: [Hardware] Add schematic frames, USB circuit, fix clocks Add schematic frames for all the different parts. Add usb connectors and associated circuity. Fix correct grounding for capacitors in the clock drivers.
Parts:
- added JP1: (no value), PortableLinuxGamestation:PINHD-1X4
- added R5: 0, PortableLinuxGamestation:R-EU_R0603
- added R6: 10k, PortableLinuxGamestation:R-EU_M0805
- added TP9: TPB1,27, PortableLinuxGamestation:TPB1,27
- added U2: FH12S-40S-0.5SH(55), PortableLinuxGamestation:FH12S-40S-0.5SH(55)
- added U3: TPD4S012, PortableLinuxGamestation:TPD4S012_DRY_6_P1_M
- added U4: MIC2287CYD5, PortableLinuxGamestation:MIC2287CYD5
- added X1: (no value), PortableLinuxGamestation:10118192-0001LF
Connections:
- new net N$22: C3.2, C4.2, U1B.OSC0_GND
- new net N$23: C1.2, C2.2, U1B.OSC1_GND
- new net N$24: R5.2, U1B.USB1_ID
- new net N$25: U1B.USB0_DM, U3.D-, X1.D-
- new net N$26: U1B.USB0_DP, U3.D+, X1.D+
- new net N$27: U1B.USB0_ID, U3.ID, X1.ID
- new net N$28: R6.2, TP9.TP, U1A.EEPROM_WP
- new net N$29: JP1.2, U1B.USB1_DM
- new net N$30: JP1.3, U1B.USB1_DP
- net EEPROM_WP: now also R6.1; no longer U1A.EEPROM_WP
- net GND: now also JP1.4, R5.1, U3.GND, X1.GND; no longer C1.2, C2.2, C3.2, C4.2
- net SYS_VOUT: now also JP1.1, U1B.USB1_VBUS
- net VDD_USB_5V: now also U1B.USB0_VBUS, U3.VBUS, X1.VBUS
Other:
- note added: "Audio"
- note added: "Clocks, ADC, USB"
- note added: "Inputs"
- note added: "LCD & Boot configuration"
- note added: "SIP Power and GND"
- note added: "Storage"
- moved on the sheet: C1, C2, C3, C4, C5, R2, R3, R4, U1B, U1C, U1D, Y1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
